Commit message: modified the base link. will add the new wheels and hitter soon

File: controller/src/rbmt_urdf/urdf/rbmt.urdf (robot description, URDF)
Before this commit: robot bot-m1, 6 links, 5 joints
Links:
- removed link omni-wheel0
- link base_link: geometry visual mesh filename=package://rbmt_urdf/mesh/Badmintonbot_versi2.stl scale=0.001 0.001 0.001
Joints:
- removed joint wheel0-joint

Commit message: added a readme for robot/main aswell as experimental .stl files

File: controller/src/rbmt_urdf/urdf/rbmt.urdf (robot description, URDF)
Before this commit: robot bot-m1, 5 links, 4 joints
Links:
- link omni-wheel1: geometry visual mesh filename=package://rbmt_urdf/mesh/Roda.stl scale=0.001 0.001 0.001

Commit message: Hopefully the robot is not in its correct position

File: controller/src/rbmt_urdf/urdf/rbmt.urdf (robot description, URDF)
Before this commit: robot bot-m1, 5 links, 4 joints
Links:
- link omni-wheel2: geometry visual mesh filename=package://rbmt_urdf/mesh/Roda.stl scale=0.001 0.001 0.001
- link omni-wheel3: geometry visual mesh filename=package://rbmt_urdf/mesh/Roda.stl scale=0.001 0.001 0.001
Joints:
- joint wheel1-joint: origin xyz=0 -0.34 0.035 rpy=0 0 1.57075 -> xyz=0.1675 0.29 0.035 rpy=0 0 1.04719
- joint wheel2-joint: origin xyz=0.294 0.17 0.035 rpy=0 0 3.665 -> xyz=-0.335 0 0.035 rpy=0 0 -3.14159
- joint wheel3-joint: origin xyz=-0.294 0.17 0.035 rpy=0 0 -0.5235 -> xyz=0.1675 -0.29 0.035 rpy=0 0 -1.04719

Commit message: URDF should now have the robot facing +X with Wheel2 aligned with X axis. robot now stands on the surface

File: controller/src/rbmt_urdf/urdf/rbmt.urdf (robot description, URDF)
Before this commit: robot bot-m1, 5 links, 4 joints
Links:
- link omni-wheel1: geometry visual mesh filename=package://rbmt_urdf/mesh/omniWheel-BIG.stl scale=0.001 0.001 0.001
- link omni-wheel2: geometry visual mesh filename=package://rbmt_urdf/mesh/omniWheel-BIG.stl scale=0.001 0.001 0.001
- link omni-wheel3: geometry visual mesh filename=package://rbmt_urdf/mesh/omniWheel-BIG.stl scale=0.001 0.001 0.001
Joints:
- joint wheel1-joint: origin xyz=0.1675 0.29 0.035 rpy=0 0 1.04719 -> xyz=0.185 0.3204 0.099 rpy=0 0 1.04719
- joint wheel2-joint: origin xyz=-0.335 0 0.035 rpy=0 0 -3.14159 -> xyz=-0.37 0 0.099 rpy=0 0 -3.14159
- joint wheel3-joint: origin xyz=0.1675 -0.29 0.035 rpy=0 0 -1.04719 -> xyz=0.185 -0.3204 0.099 rpy=0 0 -1.04719

Commit message: added .stl for hitter and positioned it to robot. added slave-rot.cc for rotation actuator of the hitter

File: controller/src/rbmt_urdf/urdf/rbmt.urdf (robot description, URDF)
Before this commit: robot bot-m1, 5 links, 4 joints
Links:
- removed link racket
- added link hitter; visual mesh filename=package://rbmt_urdf/mesh/Hitter.stl scale=0.001 0.001 0.001
Joints:
- removed joint racket_joint
- added joint roll_joint: type continuous, parent base_link, child hitter, origin xyz=0.05 -0.021 1.05 rpy=0 2.3562 0
